Commit message: add imu

File: bumperbot_description/urdf/bumperbot_base.xacro (robot description, xacro)
@@ -134,3 +134,29 @@
         <origin xyz="-0.04755 0 -0.0275" rpy="0 0 0"/>
     </joint>
+    <link name="imu_link">
+        <visual>
+            <geometry>
+                <mesh filename="package://bumperbot_description/meshes/imu_link.STL"></mesh>
+            </geometry>
+            <origin xyz="0 0 0" rpy="0 0 0"></origin>
+        </visual>
+        <collision>
+            <geometry>
+                <mesh filename="package://bumperbot_description/meshes/imu_link.STL"></mesh>
+            </geometry>
+            <origin xyz="0 0 0" rpy="0 0 0"></origin>
+        </collision>
+        <inertial>
+            <origin xyz="-0.00552433659106688 0.000168210391520346 0.000514000497342681" rpy="0 0 0" />
+            <mass value="0.000528415362211671" />
+            <inertia ixx="1.46176048428261E-08" ixy="1.40015117949421E-10" ixz="-1.99633872937403E-12"
+                     iyy="8.59662482954888E-09" iyz="7.52375112767959E-12"
+                     izz="2.30279421279312E-08" />
+          </inertial>
+    </link>
+    <joint name="base_imu_link_joint" type="fixed">
+        <parent link="base_link" />
+        <child link="imu_link" />
+        <origin xyz="0 0 0.07" rpy="0 0 0" />
+    </joint>
 </robot>

File: bumperbot_description/urdf/bumperbot_gazebo.xacro (robot description, xacro)
@@ -63,3 +63,55 @@
         </plugin>
     </gazebo>
+    <gazebo reference="imu_link">
+        <sensor name="imu" type="imu">
+            <plugin name="imu" filename="libgazebo_ros_imu_sensor.so" >
+                <topic_name>imu</topic_name>
+            </plugin>
+            <always_on>true</always_on>
+            <update_rate>100</update_rate>
+            <imu>
+                <angular_velocity>
+                    <x>
+                        <noise type="gaussian">
+                            <mean>0.0</mean>
+                            <stddev>2e-4</stddev>
+                        </noise>
+                    </x>
+                    <y>
+                        <noise type="gaussian">
+                            <mean>0.0</mean>
+                            <stddev>2e-4</stddev>
+                        </noise>
+                    </y>
+                    <z>
+                        <noise type="gaussian">
+                            <mean>0.0</mean>
+                            <stddev>2e-4</stddev>
+                        </noise>
+                    </z>
+                </angular_velocity>
+                <linear_accelration>
+                    <x>
+                        <noise type="gaussian">
+                            <mean>0.0</mean>
+                            <stddev>1.7e-2</stddev>
+                        </noise>
+                    </x>
+                    <y>
+                        <noise type="gaussian">
+                            <mean>0.0</mean>
+                            <stddev>1.7e-2</stddev>
+                        </noise>
+                    </y>
+                    <z>
+                        <noise type="gaussian">
+                            <mean>0.0</mean>
+                            <stddev>1.7e-2</stddev>
+                        </noise>
+                    </z>
+                </linear_accelration>
+            </imu>
+        </sensor>
+        <material>Gazebo/Grey</material>
+    </gazebo>
 </robot>
